File: connector/CONN-Dsub50DIL40/CONN-Dsub50DIL40.kicad_pcb (KiCad board)
At the start: 2 copper layers, 67.8 x 54.1 mm, 2 parts, among them J1 68602-140HLF, J2 D50S82C6GX00LF

Commit message: adjusted traces and added silkscreen
Other:
- board text added: "CONN-Dsub50DIL40 Lucas Darroch Brunner Neutrino Lab"
Changed lines of the file:
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@@
 		(layer "Edge.Cuts")
+	)
+	(gr_text "CONN-Dsub50DIL40\nLucas Darroch\nBrunner Neutrino Lab"
+		(at 182.16 102.97 0)
+		(layer "B.SilkS")
+		(effects
+			(font
+				(size 1 1)
+				(thickness 0.1)
+			)
+			(justify left bottom mirror)
+		)
 	)
 	(segment
